File: PCB/UMI4M.kicad_pcb (KiCad board)
At the start: 2 copper layers, 100 x 150 mm, 57 parts, among them IC1 74HCT74, IC10 74HCT08, IC11 LM7805_TO220, IC2 74HCT75, IC3 74HCT32, IC4 74HCT138, IC5 74HCT08, IC6 MC6850, IC7 MC6850, IC8 MC6850, IC9 6N137, J1 1MHzBus1, J2 1MHzBus2, J3 +5V, J4 +5V, J5 OUT 1, J6 OUT 2, J7 OUT 3, J8 IN, J9 +12V DC

Commit message: Updated
Parts:
- removed D1: MIDI 1, musix5xxx-custom:LED_D3.0mm
- removed D3: MIDI 3, musix5xxx-custom:LED_D3.0mm
- removed D6: 1N4001, Diodes_THT:D_DO-41_SOD81_P10.16mm_Horizontal
- removed the IC1 at (53.3, 41.3)
- removed the IC3 at (55.9, 97.2)
- removed the IC4 at (53.3, 73.0)
- removed IC9: 6N137, musix5xxx-custom:DIP-8_W7.62mm_LongPads
- removed the J2 at (85.0, 75.0)
- removed the J4 at (5.00, 65.0)
- removed R12, R13, R14: 220, musix5xxx-custom:R_Axial_DIN0207_L6.3mm_D2.5mm_P10.16mm_Horizontal
- added C10: C, Capacitor_THT:C_Disc_D7.5mm_W2.5mm_P5.00mm, F.Cu at (85.3, 94.6)
- added C15: C, musix5xxx-custom:C_Disc_D3.4mm_W2.1mm_P2.50mm, F.Cu at (86.4, 62.2)
- added C17: C, musix5xxx-custom:C_Disc_D3.4mm_W2.1mm_P2.50mm, F.Cu at (90.2, 72.4)
- added C4: C, Capacitor_THT:C_Disc_D7.5mm_W2.5mm_P5.00mm, F.Cu at (142.2, 66.1)
- added CD10: 0.1uF, musix5xxx-custom:C_Disc_D3.4mm_W2.1mm_P2.54mm, F.Cu at (80.0, 116.2)
- added CD11: 0.1uF, musix5xxx-custom:C_Disc_D3.4mm_W2.1mm_P2.54mm, F.Cu at (101.6, 116.2)
- added CD2: 0.1uF, musix5xxx-custom:C_Disc_D3.4mm_W2.1mm_P2.54mm, F.Cu at (204.4, 112.4)
- added CD3: 0.1uF, musix5xxx-custom:C_Disc_D3.4mm_W2.1mm_P2.54mm, F.Cu at (194.7, 63.5)
- added CD5: 0.1uF, musix5xxx-custom:C_Disc_D3.4mm_W2.1mm_P2.54mm, F.Cu at (149.8, 80.6)
- added CD7: 0.1uF, musix5xxx-custom:C_Disc_D3.4mm_W2.1mm_P2.54mm, F.Cu at (125.7, 80.0)
- added D110: 1N4148, Diode_THT:D_DO-35_SOD27_P7.62mm_Horizontal, F.Cu at (74.9, 118.1)
- added D55: 1N4148, Diode_THT:D_DO-35_SOD27_P7.62mm_Horizontal, F.Cu at (131.4, 71.1)
- added D66: 1N4001, Diode_THT:D_DO-41_SOD81_P10.16mm_Horizontal, F.Cu at (223.5, 121.9)
- added IC12: 4040, Package_DIP:DIP-16_W7.62mm_Socket_LongPads, F.Cu at (86.4, 85.1)
- added IC7: ATF22LV10C-10PU, Package_DIP:DIP-24_W7.62mm_Socket_LongPads, F.Cu at (121.9, 83.8)
- added IC8: 4001, Package_DIP:DIP-14_W7.62mm_Socket_LongPads, F.Cu at (121.3, 64.8)
- added J20: +5V, TerminalBlock_Phoenix:TerminalBlock_Phoenix_MKDS-1,5-2-5.08_1x02_P5.08mm_Horizontal, F.Cu at (78.7, 132.1)
- added J23: Conn_01x09, Connector_PinHeader_2.54mm:PinHeader_1x09_P2.54mm_Vertical, F.Cu at (173.4, 76.2)
- added J24: Conn_01x07, Connector_PinHeader_2.54mm:PinHeader_1x07_P2.54mm_Vertical, F.Cu at (96.5, 57.1)
- added J25: Conn_01x07, Connector_PinHeader_2.54mm:PinHeader_1x07_P2.54mm_Vertical, F.Cu at (76.2, 57.1)
- added J6: MULTI 1, musix5xxx-custom:din_5_pcb_mount_umi, F.Cu at (104.2, 45.7)
- added J7: MULTI 2, musix5xxx-custom:din_5_pcb_mount_umi, F.Cu at (83.8, 45.7)
- added J9: User Port, Connector_IDC:IDC-Header_2x10_P2.54mm_Vertical, F.Cu at (118.1, 123.2)
- added JP31: SolderJumper_2_Open, Jumper:SolderJumper-2_P1.3mm_Open_RoundedPad1.0x1.5mm, B.Cu at (222.9, 94.0)
- added JP32: INT TYPE, Connector_PinHeader_2.54mm:PinHeader_1x03_P2.54mm_Vertical, F.Cu at (209.6, 121.9)
- added LED1: LED, LED_THT:LED_D5.0mm, F.Cu at (147.3, 132.1)
- added OPTO1: 6N137, musix5xxx-custom:DIP-8_W7.62mm_LongPads, F.Cu at (224.8, 62.2)
- added R15: R, Resistor_THT:R_Axial_DIN0207_L6.3mm_D2.5mm_P10.16mm_Horizontal, F.Cu at (73.7, 67.3)
- added R16: R, Resistor_THT:R_Axial_DIN0207_L6.3mm_D2.5mm_P10.16mm_Horizontal, F.Cu at (73.7, 62.2)
- added R17: R, Resistor_THT:R_Axial_DIN0207_L6.3mm_D2.5mm_P10.16mm_Horizontal, F.Cu at (69.8, 77.5)
- added R18: 210R, Resistor_THT:R_Axial_DIN0207_L6.3mm_D2.5mm_P10.16mm_Horizontal, F.Cu at (134.6, 71.1)
- added R19: 120R, Resistor_THT:R_Axial_DIN0207_L6.3mm_D2.5mm_P10.16mm_Horizontal, F.Cu at (138.4, 71.1)
- added R20: 100R, Resistor_THT:R_Axial_DIN0207_L6.3mm_D2.5mm_P10.16mm_Horizontal, F.Cu at (96.5, 82.5)
- added R21: 470K, Resistor_THT:R_Axial_DIN0207_L6.3mm_D2.5mm_P10.16mm_Horizontal, F.Cu at (146.1, 71.1)
- added R22: 47?, Resistor_THT:R_Axial_DIN0207_L6.3mm_D2.5mm_P10.16mm_Horizontal, F.Cu at (101.6, 92.7)
- added R23: R, Resistor_THT:R_Axial_DIN0207_L6.3mm_D2.5mm_P10.16mm_Horizontal, F.Cu at (76.8, 91.4)
- added R24: 100R, Resistor_THT:R_Axial_DIN0207_L6.3mm_D2.5mm_P10.16mm_Horizontal, F.Cu at (98.4, 74.9)
- added R25: 100R, Resistor_THT:R_Axial_DIN0207_L6.3mm_D2.5mm_P10.16mm_Horizontal, F.Cu at (94.6, 74.9)
- added R26: R, Resistor_THT:R_Axial_DIN0207_L6.3mm_D2.5mm_P10.16mm_Horizontal, F.Cu at (90.2, 95.2)
- added R27: R, Resistor_THT:R_Axial_DIN0207_L6.3mm_D2.5mm_P10.16mm_Horizontal, F.Cu at (93.3, 113.0)
- added R28: R, Resistor_THT:R_Axial_DIN0207_L6.3mm_D2.5mm_P10.16mm_Horizontal, F.Cu at (73.7, 95.2)
- added R29: R, Resistor_THT:R_Axial_DIN0207_L6.3mm_D2.5mm_P10.16mm_Horizontal, F.Cu at (66.0, 85.1)
- added R299: R, Resistor_THT:R_Axial_DIN0207_L6.3mm_D2.5mm_P10.16mm_Horizontal, F.Cu at (102.2, 64.8)
- added R30: R, Resistor_THT:R_Axial_DIN0207_L6.3mm_D2.5mm_P10.16mm_Horizontal, F.Cu at (69.8, 85.1)
- added R31: R, Resistor_THT:R_Axial_DIN0207_L6.3mm_D2.5mm_P10.16mm_Horizontal, F.Cu at (87.0, 88.3)
- added R35: R, Resistor_THT:R_Axial_DIN0207_L6.3mm_D2.5mm_P10.16mm_Horizontal, F.Cu at (66.0, 77.5)
- added R36: 100R, Resistor_THT:R_Axial_DIN0207_L6.3mm_D2.5mm_P10.16mm_Horizontal, F.Cu at (71.1, 105.4)
- added R37: 100R, Resistor_THT:R_Axial_DIN0207_L6.3mm_D2.5mm_P10.16mm_Horizontal, F.Cu at (67.3, 105.4)
- added R555: 1K, Resistor_THT:R_Axial_DIN0207_L6.3mm_D2.5mm_P10.16mm_Horizontal, F.Cu at (127.0, 129.5)
- added R666: 10K, Resistor_THT:R_Axial_DIN0207_L6.3mm_D2.5mm_P10.16mm_Horizontal, F.Cu at (228.6, 61.0)
- added REF**: KiCad-Logo2_6mm_SilkScreen, Symbol:KiCad-Logo2_6mm_SilkScreen, F.Cu at (142.9, 112.4)
- added REG1: LM7805_TO220, Package_TO_SOT_THT:TO-220-3_Vertical, F.Cu at (236.2, 119.4)
- added TP1: CNPGFC, TestPoint:TestPoint_THTPad_D2.0mm_Drill1.0mm, F.Cu at (132.7, 107.3)
- added TP3: 3, TestPoint:TestPoint_THTPad_D2.0mm_Drill1.0mm, F.Cu at (190.5, 56.5)
- added TP4: 4, TestPoint:TestPoint_THTPad_D2.0mm_Drill1.0mm, F.Cu at (170.2, 56.5)
- added TP5: 5, TestPoint:TestPoint_THTPad_D2.0mm_Drill1.0mm, F.Cu at (143.5, 56.5)
- added TP6: 6, TestPoint:TestPoint_THTPad_D2.0mm_Drill1.0mm, F.Cu at (119.4, 53.3)
- added U7: 4050, Package_DIP:DIP-16_W7.62mm_LongPads, F.Cu at (191.1, 63.5)
- C1: value 220pF -> C_Polarized; footprint musix5xxx-custom:C_Disc_D3.4mm_W2.1mm_P2.50mm -> Capacitor_THT:CP_Radial_Tantal_D4.5mm_P2.50mm
- C11: footprint musix5xxx-custom:CP_Radial_D6.3mm_P2.50mm -> Capacitor_THT:CP_Radial_D5.0mm_P2.00mm
- C12, C2: footprint musix5xxx-custom:CP_Radial_D6.3mm_P2.50mm -> Capacitor_THT:CP_Radial_D5.0mm_P2.50mm
- C3, C8, C9: value 0.1uF -> C; footprint musix5xxx-custom:C_Disc_D3.4mm_W2.1mm_P2.50mm -> Capacitor_THT:C_Disc_D7.5mm_W2.5mm_P5.00mm
- C6, C7: value 0.1uF -> C
- CD1: renamed from C10; footprint musix5xxx-custom:C_Disc_D3.4mm_W2.1mm_P2.50mm -> musix5xxx-custom:C_Disc_D3.4mm_W2.1mm_P2.54mm
- CD4: renamed from C4; footprint musix5xxx-custom:C_Disc_D3.4mm_W2.1mm_P2.50mm -> musix5xxx-custom:C_Disc_D3.4mm_W2.1mm_P2.54mm
- CD8: renamed from C5; footprint musix5xxx-custom:C_Disc_D3.4mm_W2.1mm_P2.50mm -> musix5xxx-custom:C_Disc_D3.4mm_W2.1mm_P2.54mm
- D2: value MIDI 2 -> 1N4148; footprint musix5xxx-custom:LED_D3.0mm -> Diode_THT:D_DO-35_SOD27_P7.62mm_Horizontal
- D4: value PWR -> 1N4148; footprint musix5xxx-custom:LED_D3.0mm -> Diode_THT:D_DO-35_SOD27_P7.62mm_Horizontal
- D5: value 4148 -> 1N4148; footprint musix5xxx-custom:D_DO-35_SOD27_P10.16mm_Horizontal -> Diode_THT:D_DO-35_SOD27_P7.62mm_Horizontal
- D7: value MIDI 3 in -> 1N4148; footprint musix5xxx-custom:LED_D3.0mm -> Diode_THT:D_DO-35_SOD27_P7.62mm_Horizontal
- H1, H2, H3, H4: value 3.5mm -> MountingHole; footprint Mounting_Holes:MountingHole_3.5mm_Pad -> MountingHole:MountingHole_4.3mm_M4
- IC1: renamed from IC8; footprint musix5xxx-custom:DIP-24_W15.24mm_LongPads -> Package_DIP:DIP-24_W15.24mm_Socket_LongPads
- IC10: value 74HCT08 -> 4066; footprint musix5xxx-custom:DIP-14_W7.62mm_LongPads -> Package_DIP:DIP-14_W7.62mm_Socket_LongPads
- IC11: value LM7805_TO220 -> HEF4093B; footprint TO_SOT_Packages_THT:TO-220-3_Vertical -> Package_DIP:DIP-14_W7.62mm_Socket_LongPads
- IC2: value 74HCT75 -> MC6850; footprint musix5xxx-custom:DIP-16_W7.62mm_LongPads -> Package_DIP:DIP-24_W15.24mm_Socket_LongPads
- IC3: renamed from IC7; footprint musix5xxx-custom:DIP-24_W15.24mm_LongPads -> Package_DIP:DIP-24_W15.24mm_Socket_LongPads
- IC4: renamed from IC6; footprint musix5xxx-custom:DIP-24_W15.24mm_LongPads -> Package_DIP:DIP-24_W15.24mm_Socket_LongPads
- IC5: value 74HCT08 -> ATF16V8; footprint musix5xxx-custom:DIP-14_W7.62mm_LongPads -> Package_DIP:DIP-20_W7.62mm_LongPads
- J1: renamed from J8; value IN -> IN 1; footprint musix5xxx-custom:din_5_pcb_mount -> musix5xxx-custom:din_5_pcb_mount_umi
- J2: renamed from J7; value OUT 3 -> OUT 1; footprint musix5xxx-custom:din_5_pcb_mount -> musix5xxx-custom:din_5_pcb_mount_umi
- J21: renamed from J9; footprint Connectors_Molex:Molex_KK-6410-02_02x2.54mm_Straight -> TerminalBlock_Phoenix:TerminalBlock_Phoenix_MKDS-1,5-2-5.08_1x02_P5.08mm_Horizontal
- J3: value +5V -> OUT 2; footprint musix5xxx-custom:Molex_KK-6410-02_02x2.54mm_Straight -> musix5xxx-custom:din_5_pcb_mount_umi
- J4: renamed from J6; value OUT 2 -> OUT 3; footprint musix5xxx-custom:din_5_pcb_mount -> musix5xxx-custom:din_5_pcb_mount_umi
- J5: value OUT 1 -> OUT 4; footprint musix5xxx-custom:din_5_pcb_mount -> musix5xxx-custom:din_5_pcb_mount_umi
- J8: renamed from J1; footprint musix5xxx-custom:IDC-Header_2x17_Pitch2.54mm_Angled -> Connector_IDC:IDC-Header_2x17_P2.54mm_Vertical
- R1, R8, R9: footprint musix5xxx-custom:R_Axial_DIN0207_L6.3mm_D2.5mm_P10.16mm_Horizontal -> Resistor_THT:R_Axial_DIN0207_L6.3mm_D2.5mm_P10.16mm_Horizontal
- R10: value 220 -> 680R; footprint musix5xxx-custom:R_Axial_DIN0207_L6.3mm_D2.5mm_P10.16mm_Horizontal -> Resistor_THT:R_Axial_DIN0207_L6.3mm_D2.5mm_P10.16mm_Horizontal
- R11: value 220 -> 470K; footprint musix5xxx-custom:R_Axial_DIN0207_L6.3mm_D2.5mm_P10.16mm_Horizontal -> Resistor_THT:R_Axial_DIN0207_L6.3mm_D2.5mm_P10.16mm_Horizontal
- R2, R3, R4, R7: value 330 -> 220; footprint musix5xxx-custom:R_Axial_DIN0207_L6.3mm_D2.5mm_P10.16mm_Horizontal -> Resistor_THT:R_Axial_DIN0207_L6.3mm_D2.5mm_P10.16mm_Horizontal
- R5: value 1K -> 220; footprint musix5xxx-custom:R_Axial_DIN0207_L6.3mm_D2.5mm_P10.16mm_Horizontal -> Resistor_THT:R_Axial_DIN0207_L6.3mm_D2.5mm_P10.16mm_Horizontal
- R6: value 10K -> 220; footprint musix5xxx-custom:R_Axial_DIN0207_L6.3mm_D2.5mm_P10.16mm_Horizontal -> Resistor_THT:R_Axial_DIN0207_L6.3mm_D2.5mm_P10.16mm_Horizontal
- moved J21 236.6 mm to (215.9, 129.5), turned to 0 degrees
- moved IC1 228.2 mm to (231.1, 109.2), turned to 180 degrees
- moved C2 223.4 mm to (229.9, 113.1), turned to -90 degrees
- moved C11 220.8 mm to (229.9, 121.4), turned to 90 degrees
- moved R5 199.6 mm to (201.9, 71.1), turned to 90 degrees
- moved R2 198.4 mm to (205.7, 71.1), turned to 90 degrees
- moved CD1 198.0 mm to (224.8, 112.4), turned to 180 degrees
- moved R3 197.8 mm to (209.6, 71.1), turned to 90 degrees
- moved R4 182.4 mm to (198.1, 71.1), turned to 90 degrees
- moved IC3 180.8 mm to (190.5, 109.2), turned to 180 degrees
- moved J3 170.3 mm to (172.7, 45.7), turned to 0 degrees
- moved IC2 165.7 mm to (210.8, 109.2), turned to 180 degrees
- moved R1 162.3 mm to (236.2, 71.1)
- moved R10 157.9 mm to (213.4, 71.1), turned to 90 degrees
- moved IC4 156.9 mm to (170.2, 109.2), turned to 180 degrees
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Connections:
- C1 pad 1: +5V -> EXT_CLK_IN
- C1 pad 2: Net-(C1-Pad2) -> Net-(D2-A)
- C11 pad 1: Net-(C11-Pad1) -> /12VD
- C3 pad 1: +5V -> Net-(C3-Pad1)
- C3 pad 2: GND -> FOOTSWITCH
- C6 pad 1: +5V -> Net-(C6-Pad1)
- C6 pad 2: GND -> CLOCK_OUT
- C7 pad 1: +5V -> Net-(C7-Pad1)
- C8 pad 1: +5V -> Net-(IC12-Q9)
- C8 pad 2: GND -> Net-(C8-Pad2)
- C9 pad 1: +5V -> Net-(C9-Pad1)
- C9 pad 2: GND -> START_CON
- D2 pad 1: Net-(D2-Pad1) -> Y3
- D2 pad 2: +5V -> Net-(D2-A)
- D4 pad 1: GND -> Net-(D110-A)
- D4 pad 2: Net-(D4-Pad2) -> GND
- D5 pad 1: Net-(D5-Pad1) -> Y4
- D5 pad 2: Net-(D5-Pad2) -> Net-(D5-A)
- D7 pad 1: Net-(D7-Pad1) -> Net-(D7-K)
- D7 pad 2: +5V -> Net-(D7-A)
- IC1 pad 11: /a0 -> /A0
- IC1 pad 13: R~W~' -> R~{W}B
- IC1 pad 15: /d7 -> /D7
- IC1 pad 16: /d6 -> /D6
- IC1 pad 17: /d5 -> /D5
- IC1 pad 18: /d4 -> /D4
- IC1 pad 19: /d3 -> /D3
- IC1 pad 2: RX3 -> RX1
- IC1 pad 20: /d2 -> /D2
- IC1 pad 21: /d1 -> /D1
- IC1 pad 22: /d0 -> /D0
- IC1 pad 3: CLK-6850 -> SER_CLK
- IC1 pad 4: CLK-6850 -> SER_CLK
- IC1 pad 5: Net-(IC8-Pad5) -> unconnected-(IC1-~{RTS}-Pad5)
- IC1 pad 6: TX3 -> TX1
- IC1 pad 7: /~IRQ -> ~{INT}
- IC1 pad 9: CS2-3 -> CS_A
- IC10 pad 1: TX1 -> Net-(IC12-Q0)
- IC10 pad 10: TX3 -> /Untitled Sheet/PB0
- IC10 pad 11: Net-(IC10-Pad11) -> GND
- IC10 pad 12: RX3 -> Net-(IC10-Pad12)
- IC10 pad 13: RX3 -> /Untitled Sheet/PB4
- IC10 pad 2: TX1 -> Net-(IC10-Pad2)
- IC10 pad 3: Net-(IC10-Pad3) -> Net-(IC12-Q0)
- IC10 pad 4: TX2 -> Net-(D110-A)
- IC10 pad 5: TX2 -> /Untitled Sheet/PB5
- IC10 pad 6: Net-(IC10-Pad6) -> GND
- IC10 pad 8: Net-(IC10-Pad8) -> unconnected-(IC10-Pad8)
- IC10 pad 9: TX3 -> unconnected-(IC10-Pad9)
- IC11 pad 1: Net-(C11-Pad1) -> +5V
- IC11 pad 2: GND -> Net-(IC12-Q0)
- IC11 pad 3: +5V -> /Untitled Sheet/PB6
- IC2 pad 1: Net-(IC2-Pad1) -> GND
- IC2 pad 10: CP2-1 -> +5V
- IC2 pad 11: Net-(IC2-Pad11) -> /A0
- IC2 pad 12: GND -> +5V
- IC2 pad 13: Net-(IC2-Pad11) -> R~{W}B
- IC2 pad 14: Net-(IC2-Pad14) -> /1MHZE
- IC2 pad 15: Net-(IC2-Pad15) -> /D7
- IC2 pad 16: Net-(IC2-Pad16) -> /D6
- IC2 pad 2: /~PGFC -> GND
- IC2 pad 3: +5V -> SER_CLK
- IC2 pad 4: +5V -> SER_CLK
- IC2 pad 5: +5V -> unconnected-(IC2-~{RTS}-Pad5)
- IC2 pad 6: /1MHZE -> TX2
- IC2 pad 7: +5V -> ~{INT2}
- IC2 pad 8: Net-(IC2-Pad8) -> +5V
- IC2 pad 9: Net-(IC2-Pad9) -> CS_B
- IC3 pad 11: /a0 -> /A0
- IC3 pad 13: R~W~' -> R~{W}B
- IC3 pad 15: /d7 -> /D7
- IC3 pad 16: /d6 -> /D6
- IC3 pad 17: /d5 -> /D5
- IC3 pad 18: /d4 -> /D4
- IC3 pad 19: /d3 -> /D3
- IC3 pad 20: /d2 -> /D2
- IC3 pad 21: /d1 -> /D1
- IC3 pad 22: /d0 -> /D0
- IC3 pad 3: CLK-6850 -> SER_CLK
- IC3 pad 4: CLK-6850 -> SER_CLK
- IC3 pad 5: Net-(IC7-Pad5) -> unconnected-(IC3-~{RTS}-Pad5)
- IC3 pad 6: TX2 -> TX3
- IC3 pad 7: /~IRQ -> ~{INT2}
- IC3 pad 9: CS2-2 -> CS_C
- IC4 pad 11: /a0 -> /A0
- IC4 pad 13: R~W~' -> R~{W}B
- IC4 pad 15: /d7 -> /D7
- IC4 pad 16: /d6 -> /D6
- IC4 pad 17: /d5 -> /D5
- IC4 pad 18: /d4 -> /D4
- IC4 pad 19: /d3 -> /D3
- IC4 pad 20: /d2 -> /D2
- IC4 pad 21: /d1 -> /D1
- IC4 pad 22: /d0 -> /D0
- IC4 pad 3: CLK-6850 -> SER_CLK
- IC4 pad 4: CLK-6850 -> SER_CLK
- IC4 pad 5: Net-(IC6-Pad5) -> unconnected-(IC4-~{RTS}-Pad5)
- IC4 pad 6: TX1 -> TX4
- IC4 pad 7: /~IRQ -> ~{INT2}
- IC4 pad 9: CS2-1 -> CS_D
- IC5 pad 1: TX1 -> unconnected-(IC5-I1/CLK-Pad1)
- IC5 pad 10: TX3 -> GND
- IC5 pad 11: Net-(IC5-Pad11) -> CS_ID
- IC5 pad 12: GND -> /D0
- IC5 pad 13: GND -> /D1
- IC5 pad 14: +5V -> /D2
- IC5 pad 2: TX1 -> /A0
- IC5 pad 3: Net-(IC5-Pad3) -> /A1
- IC5 pad 4: TX2 -> /A2
- IC5 pad 5: TX2 -> /A3
- IC5 pad 6: Net-(IC5-Pad6) -> /A4
- IC5 pad 7: GND -> unconnected-(IC5-I7-Pad7)
- IC5 pad 8: Net-(IC5-Pad8) -> unconnected-(IC5-I8-Pad8)
- IC5 pad 9: TX3 -> unconnected-(IC5-I9-Pad9)
- J1 pad 1: Net-(J8-Pad1) -> unconnected-(J1-Pad1)
- J1 pad 2: Net-(J8-Pad2) -> unconnected-(J1-Pad2)
- J1 pad 3: Net-(J8-Pad3) -> unconnected-(J1-Pad3)
- J1 pad 4: Net-(J8-Pad4) -> Net-(J1-Pad4)
- J1 pad 5: Net-(D5-Pad2) -> Net-(D7-A)
- J1 pad S1: (no net) -> unconnected-(J1-PadS1)_3
- J2 pad 1: Net-(J7-Pad1) -> unconnected-(J2-Pad1)
- J2 pad 3: Net-(J7-Pad3) -> unconnected-(J2-Pad3)
- J2 pad 4: Net-(J7-Pad4) -> Net-(J2-Pad4)
- J2 pad 5: Net-(J7-Pad5) -> Net-(J2-Pad5)
- J2 pad S1: (no net) -> unconnected-(J2-PadS1)_3
- J21 pad 1: Net-(D6-Pad2) -> +12V
- J3 pad 1: +5V -> Net-(J3-Pad1)
- J4 pad 1: Net-(J6-Pad1) -> unconnected-(J4-Pad1)
- J4 pad 3: Net-(J6-Pad3) -> unconnected-(J4-Pad3)
- J4 pad 4: Net-(J6-Pad4) -> Net-(J4-Pad4)
- J4 pad 5: Net-(J6-Pad5) -> Net-(J4-Pad5)
- J4 pad S1: (no net) -> unconnected-(J4-PadS1)_3
- J5 pad S1: (no net) -> unconnected-(J5-PadS1)_3
- J8 pad 10: /~PGFC -> /~{PGFC}
- J8 pad 12: /~PGFD -> /~{PGFD}
- J8 pad 14: /~RST -> /~{RST}
- J8 pad 16: /AUDIO -> AUDIO
- J8 pad 18: /d0 -> /D0
- J8 pad 19: /d1 -> /D1
- J8 pad 2: /R~W -> /R~{W}
- J8 pad 20: /d2 -> /D2
- J8 pad 21: /d3 -> /D3
- J8 pad 22: /d4 -> /D4
- J8 pad 23: /d5 -> /D5
- J8 pad 24: /d6 -> /D6
- J8 pad 25: /d7 -> /D7
- J8 pad 27: /a0 -> /A0
- J8 pad 28: /a1 -> /A1
- J8 pad 29: /a2 -> /A2
- J8 pad 30: /a3 -> /A3
- J8 pad 31: /a4 -> /A4
- J8 pad 32: /a5 -> /A5
- J8 pad 33: /a6 -> /A6
- J8 pad 34: /a7 -> /A7
- J8 pad 6: /~NMI -> /~{NMI}
- J8 pad 8: /~IRQ -> /~{IRQ}
- R1 pad 1: Net-(IC1-Pad8) -> Net-(D7-K)
- R1 pad 2: Net-(C1-Pad2) -> Net-(J1-Pad4)
- R10 pad 2: Net-(J6-Pad4) -> RX1
- R11 pad 1: Net-(IC5-Pad6) -> +5V
- R11 pad 2: Net-(J6-Pad5) -> Net-(D2-A)
- R2 pad 1: Net-(IC10-Pad3) -> +5V
- R2 pad 2: Net-(D1-Pad1) -> Net-(J2-Pad4)
- R3 pad 1: Net-(IC10-Pad6) -> Net-(R3-Pad1)
- R3 pad 2: Net-(D2-Pad1) -> Net-(J2-Pad5)
- R4 pad 1: Net-(IC10-Pad8) -> +5V
- R4 pad 2: Net-(D3-Pad1) -> Net-(J3-Pad4)
- R5 pad 1: +5V -> Net-(R5-Pad1)
- R5 pad 2: Net-(D4-Pad2) -> Net-(J3-Pad5)
- R6 pad 1: RX3 -> +5V
- R6 pad 2: +5V -> Net-(J4-Pad4)
- R7 pad 1: Net-(IC10-Pad11) -> Net-(R7-Pad1)
- R7 pad 2: Net-(D7-Pad1) -> Net-(J4-Pad5)
- R9 pad 1: Net-(IC5-Pad3) -> Net-(R9-Pad1)
Routing:
- net GND: track 106.0 -> 1105.1 mm
- net /d0: track 187.9 -> 0.00 mm, vias 1 -> 0
- net RX3: track 165.7 -> 0.00 mm, vias 1 -> 0
- net CS_A: track 0.00 -> 162.7 mm, vias 0 -> 3
- net /A0: track 0.00 -> 155.0 mm, vias 0 -> 2
- net CLK-6850: track 153.9 -> 0.00 mm, vias 1 -> 0
- net /d2: track 142.5 -> 0.00 mm
- net /d1: track 142.4 -> 0.00 mm
- net /~IRQ: track 137.9 -> 0.00 mm, vias 1 -> 0
- net AUDIO: track 0.00 -> 137.0 mm, vias 0 -> 1
- net /d4: track 136.4 -> 0.00 mm
- net /d3: track 136.3 -> 0.00 mm
- net CS_B: track 0.00 -> 135.2 mm, vias 0 -> 3
- net /a0: track 131.2 -> 0.00 mm, vias 1 -> 0
- net /d6: track 130.9 -> 0.00 mm
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- removed copper zone on B.Cu, net GND
- removed copper zone on F.Cu, net GND
Other:
- board size 100 x 150 mm -> 176.8 x 100.3 mm
- net class Default removed
- net class PWR removed
- net class bus removed
- board text added: "POWER"
- board text added: "See https://github.com/fordp2002/music2xxx"
- board text added: "Universal MIDI Interface"
- board text added: "User Port"
- board text removed: "1"
- board text removed: "2"
- board text removed: "3"
- board text removed: "5V GND"
- board text removed: "Based on Hybrid M2000 Midi Interface This PCB and mods by J Lane September 2019"
- board text removed: "Music 2xxx Midi Interface"
