File: PCB/UMI4M.kicad_sch (KiCad schematic)
At the start: 57 parts, among them IC1 74HCT74, IC10 74HCT08, IC101 MC6850, IC11 LM7805_TO220, IC12 MC6850, IC2 74HCT75, IC3 74HCT32, IC4 74HCT138, IC5 74HCT08, IC6 MC6850, IC7 MC6850, IC8 74HCT08, IC9 6N137, J102 OUT 1, J103 OUT 2, J104 OUT 3, J105 OUT 4, J3 +5V, J8 1MHzBus1, J8 IN 1, J9 +12V DC

Commit message: Updated
Parts:
- removed C1: 220pF, musix5xxx-custom:C_Disc_D3.4mm_W2.1mm_P2.50mm, symbol Device:C
- removed D2, D3, D4, D5: LED, symbol Device:LED
- removed IC1: 74HCT74, musix5xxx-custom:DIP-14_W7.62mm_LongPads, symbol 74xx:74LS74
- removed IC10, IC5, IC8: 74HCT08, musix5xxx-custom:DIP-14_W7.62mm_LongPads, symbol 74xx:74LS08
- removed IC11: LM7805_TO220, TO_SOT_Packages_THT:TO-220-3_Vertical, symbol Regulator_Linear:LM7805_TO220
- removed IC2: 74HCT75, musix5xxx-custom:DIP-16_W7.62mm_LongPads, symbol 74xx:74LS75
- removed IC3: 74HCT32, musix5xxx-custom:DIP-14_W7.62mm_LongPads, symbol 74xx:74LS32
- removed IC4: 74HCT138, musix5xxx-custom:DIP-16_W7.62mm_LongPads, symbol 74xx:74LS138
- removed R1: 220, musix5xxx-custom:R_Axial_DIN0207_L6.3mm_D2.5mm_P10.16mm_Horizontal, symbol Device:R
- removed R2, R3, R4, R7: 330, musix5xxx-custom:R_Axial_DIN0207_L6.3mm_D2.5mm_P10.16mm_Horizontal, symbol Device:R
- added CD3: 0.1uF, musix5xxx-custom:C_Disc_D3.4mm_W2.1mm_P2.54mm, symbol Device:C
- added H1, H2, H3, H4: MountingHole, MountingHole:MountingHole_4.3mm_M4, symbol Mechanical:MountingHole
- added IC5: ATF16V8, Package_DIP:DIP-20_W7.62mm_LongPads, symbol Logic_Programmable:GAL16V8
- added IC7: ATF22LV10C-10PU, Package_DIP:DIP-24_W7.62mm_Socket_LongPads, symbol 2025-03-10_10-04-24:ATF22LV10C-10PU
- added J23: Conn_01x09, Connector_PinHeader_2.54mm:PinHeader_1x09_P2.54mm_Vertical, symbol Connector_Generic:Conn_01x09
- added JP31: SolderJumper_2_Open, Jumper:SolderJumper-2_P1.3mm_Open_RoundedPad1.0x1.5mm, symbol Jumper:SolderJumper_2_Open
- added R10: 680R, Resistor_THT:R_Axial_DIN0207_L6.3mm_D2.5mm_P10.16mm_Horizontal, symbol Device:R
- added REG1: LM7805_TO220, Package_TO_SOT_THT:TO-220-3_Vertical, symbol Regulator_Linear:LM7805_TO220
- added TP1: CNPGFC, TestPoint:TestPoint_THTPad_D2.0mm_Drill1.0mm, symbol Connector:TestPoint
- added TP3: 3, TestPoint:TestPoint_THTPad_D2.0mm_Drill1.0mm, symbol Connector:TestPoint
- added TP4: 4, TestPoint:TestPoint_THTPad_D2.0mm_Drill1.0mm, symbol Connector:TestPoint
- added TP5: 5, TestPoint:TestPoint_THTPad_D2.0mm_Drill1.0mm, symbol Connector:TestPoint
- added TP6: 6, TestPoint:TestPoint_THTPad_D2.0mm_Drill1.0mm, symbol Connector:TestPoint
- added U7: 4050, Package_DIP:DIP-16_W7.62mm_LongPads, symbol 4xxx:4050
- C11: footprint (none) -> Capacitor_THT:CP_Radial_D5.0mm_P2.00mm
- C12, C2: footprint (none) -> Capacitor_THT:CP_Radial_D5.0mm_P2.50mm
- CD1: renamed from C10; footprint musix5xxx-custom:C_Disc_D3.4mm_W2.1mm_P2.50mm -> musix5xxx-custom:C_Disc_D3.4mm_W2.1mm_P2.54mm
- CD10: renamed from C7; footprint musix5xxx-custom:C_Disc_D3.4mm_W2.1mm_P2.50mm -> musix5xxx-custom:C_Disc_D3.4mm_W2.1mm_P2.54mm
- CD11: renamed from C8; footprint musix5xxx-custom:C_Disc_D3.4mm_W2.1mm_P2.50mm -> musix5xxx-custom:C_Disc_D3.4mm_W2.1mm_P2.54mm
- CD2: renamed from C3; footprint musix5xxx-custom:C_Disc_D3.4mm_W2.1mm_P2.50mm -> musix5xxx-custom:C_Disc_D3.4mm_W2.1mm_P2.54mm
- CD4: renamed from C4; footprint musix5xxx-custom:C_Disc_D3.4mm_W2.1mm_P2.50mm -> musix5xxx-custom:C_Disc_D3.4mm_W2.1mm_P2.54mm
- CD5: renamed from C6; footprint musix5xxx-custom:C_Disc_D3.4mm_W2.1mm_P2.50mm -> musix5xxx-custom:C_Disc_D3.4mm_W2.1mm_P2.54mm
- CD7: renamed from C9; footprint musix5xxx-custom:C_Disc_D3.4mm_W2.1mm_P2.50mm -> musix5xxx-custom:C_Disc_D3.4mm_W2.1mm_P2.54mm
- CD8: renamed from C5; footprint musix5xxx-custom:C_Disc_D3.4mm_W2.1mm_P2.50mm -> musix5xxx-custom:C_Disc_D3.4mm_W2.1mm_P2.54mm
- D66: renamed from D6; footprint Diodes_THT:D_DO-41_SOD81_P10.16mm_Horizontal -> Diode_THT:D_DO-41_SOD81_P10.16mm_Horizontal
- IC1: renamed from IC101; footprint musix5xxx-custom:DIP-24_W15.24mm_LongPads -> Package_DIP:DIP-24_W15.24mm_Socket_LongPads
- IC2: renamed from IC12; footprint musix5xxx-custom:DIP-24_W15.24mm_LongPads -> Package_DIP:DIP-24_W15.24mm_Socket_LongPads
- IC3: renamed from IC7; footprint musix5xxx-custom:DIP-24_W15.24mm_LongPads -> Package_DIP:DIP-24_W15.24mm_Socket_LongPads
- IC4: renamed from IC6; footprint musix5xxx-custom:DIP-24_W15.24mm_LongPads -> Package_DIP:DIP-24_W15.24mm_Socket_LongPads
- J1: renamed from J8; footprint musix5xxx-custom:din_5_pcb_mount -> musix5xxx-custom:din_5_pcb_mount_umi; symbol Connector:DIN-5_180degree -> music5xxx-custom:DIN-5_180degree
- J2: renamed from J102; footprint musix5xxx-custom:din_5_pcb_mount -> musix5xxx-custom:din_5_pcb_mount_umi; symbol Connector:DIN-5_180degree -> music5xxx-custom:DIN-5_180degree
- J20: renamed from J3; footprint Connectors_Molex:Molex_KK-6410-02_02x2.54mm_Straight -> TerminalBlock_Phoenix:TerminalBlock_Phoenix_MKDS-1,5-2-5.08_1x02_P5.08mm_Horizontal
- J21: renamed from J9; footprint Connectors_Molex:Molex_KK-6410-02_02x2.54mm_Straight -> TerminalBlock_Phoenix:TerminalBlock_Phoenix_MKDS-1,5-2-5.08_1x02_P5.08mm_Horizontal
- J3: renamed from J103; footprint musix5xxx-custom:din_5_pcb_mount -> musix5xxx-custom:din_5_pcb_mount_umi; symbol Connector:DIN-5_180degree -> music5xxx-custom:DIN-5_180degree
- J4: renamed from J104; footprint musix5xxx-custom:din_5_pcb_mount -> musix5xxx-custom:din_5_pcb_mount_umi; symbol Connector:DIN-5_180degree -> music5xxx-custom:DIN-5_180degree
- J5: renamed from J105; footprint musix5xxx-custom:din_5_pcb_mount -> musix5xxx-custom:din_5_pcb_mount_umi; symbol Connector:DIN-5_180degree -> music5xxx-custom:DIN-5_180degree
- J8: footprint musix5xxx-custom:IDC-Header_2x17_Pitch2.54mm_Angled -> Connector_IDC:IDC-Header_2x17_P2.54mm_Vertical
- JP32: renamed from JP1; footprint (none) -> Connector_PinHeader_2.54mm:PinHeader_1x03_P2.54mm_Vertical
- LED1: renamed from D7; footprint (none) -> LED_THT:LED_D5.0mm
- R1: renamed from R14; footprint musix5xxx-custom:R_Axial_DIN0207_L6.3mm_D2.5mm_P10.16mm_Horizontal -> Resistor_THT:R_Axial_DIN0207_L6.3mm_D2.5mm_P10.16mm_Horizontal
- R2: renamed from R12; footprint musix5xxx-custom:R_Axial_DIN0207_L6.3mm_D2.5mm_P10.16mm_Horizontal -> Resistor_THT:R_Axial_DIN0207_L6.3mm_D2.5mm_P10.16mm_Horizontal
- R3: renamed from R13; footprint musix5xxx-custom:R_Axial_DIN0207_L6.3mm_D2.5mm_P10.16mm_Horizontal -> Resistor_THT:R_Axial_DIN0207_L6.3mm_D2.5mm_P10.16mm_Horizontal
- R4: renamed from R15; footprint musix5xxx-custom:R_Axial_DIN0207_L6.3mm_D2.5mm_P10.16mm_Horizontal -> Resistor_THT:R_Axial_DIN0207_L6.3mm_D2.5mm_P10.16mm_Horizontal
- R5: renamed from R16; footprint musix5xxx-custom:R_Axial_DIN0207_L6.3mm_D2.5mm_P10.16mm_Horizontal -> Resistor_THT:R_Axial_DIN0207_L6.3mm_D2.5mm_P10.16mm_Horizontal
- R555: renamed from R5; footprint musix5xxx-custom:R_Axial_DIN0207_L6.3mm_D2.5mm_P10.16mm_Horizontal -> Resistor_THT:R_Axial_DIN0207_L6.3mm_D2.5mm_P10.16mm_Horizontal
- R6: renamed from R10; footprint musix5xxx-custom:R_Axial_DIN0207_L6.3mm_D2.5mm_P10.16mm_Horizontal -> Resistor_THT:R_Axial_DIN0207_L6.3mm_D2.5mm_P10.16mm_Horizontal
- R666: renamed from R6; footprint musix5xxx-custom:R_Axial_DIN0207_L6.3mm_D2.5mm_P10.16mm_Horizontal -> Resistor_THT:R_Axial_DIN0207_L6.3mm_D2.5mm_P10.16mm_Horizontal
- R7: renamed from R11; footprint musix5xxx-custom:R_Axial_DIN0207_L6.3mm_D2.5mm_P10.16mm_Horizontal -> Resistor_THT:R_Axial_DIN0207_L6.3mm_D2.5mm_P10.16mm_Horizontal
- R8, R9: footprint musix5xxx-custom:R_Axial_DIN0207_L6.3mm_D2.5mm_P10.16mm_Horizontal -> Resistor_THT:R_Axial_DIN0207_L6.3mm_D2.5mm_P10.16mm_Horizontal
- renumbered D1 to D7, IC9 to OPTO1
Connections:
- net 0V is gone; now on net GND: J8.1 (Pin_1), J8.11 (Pin_11), J8.13 (Pin_13), J8.15 (Pin_15), J8.17 (Pin_17), J8.26 (Pin_26), J8.3 (Pin_3), J8.5 (Pin_5), J8.7 (Pin_7), J8.9 (Pin_9)
- net +5V: now also IC2.10 (CS1), IC2.8 (CS0), CD3.1, IC5.20 (VCC), IC7.24 (VCC), J23.9 (Pin_9), R10.1, REG1.3 (VO), U7.1 (VCC); no longer OPTO1.8, R666.2
- net 1MHZE: now also IC2.14 (E), IC7.1 (CLK/IN)
- net CS_A: now also IC7.23 (I/O)
- net CS_B: now also IC7.22 (I/O)
- net CS_C: now also IC7.18 (I/O)
- net CS_D: now also IC7.17 (I/O)
- net GND: now also IC1.1 (VSS), IC2.1 (VSS), IC3.1 (VSS), CD3.2, IC5.10 (GND), IC7.12 (GND), J23.1 (Pin_1), REG1.2 (GND), U7.8 (VSS); no longer IC1.2 (Rx_Data)
- net R~{W}: now also IC7.11 (IN)
- net SER_CLK: now also IC2.3 (Rx_CLK), IC2.4 (Tx_CLK), IC7.14 (I/O)
- net TX1: now also J23.7 (Pin_7), U7.3
- net TX2: now also IC2.6 (Tx_Data), J23.5 (Pin_5), J23.6 (Pin_6), U7.14
- net TX3: now also J23.3 (Pin_3), J23.4 (Pin_4), U7.9
- net TX4: now also J23.2 (Pin_2), U7.11
- net ~{INT}: now also JP31.1 (A); no longer IC2.7 (~{IRQ}), IC3.7 (~{IRQ}), IC4.7 (~{IRQ})
- net ~{IRQ}: now also JP32.3 (B); no longer JP32.1 (A)
- net ~{NMI}: now also JP32.1 (A); no longer JP32.3 (B)
- net ~{PGFC}: now also IC7.10 (IN)
- net ~{PGFD}: now also IC7.13 (IN)
- net at R7.1: now also U7.10
- net at R3.1: now also U7.2
- net RX1: now reaches OPTO1.6, R666.1
- net RX1: now also IC1.2 (Rx_Data), J23.8 (Pin_8), R10.2
- net at R9.1: now also U7.12
- net at J5.1: now also TP6.1
- net at J5.3: now also TP5.1
- net 12VD: now reaches C11.1, D66.1 (K)
- net 12VD: now also REG1.1 (VI)
- net +12V: now reaches D66.2 (A), J21.1 (Pin_1)
- net at R5.1: now also U7.15
- net at J3.1: now also TP4.1
- net at J3.3: now also TP3.1
- net R~{W}' renamed R~{W}B
- net R~{W}B: now also IC7.21 (I/O)
- net a0 renamed A0
- net A0: now also IC5.2 (I2), IC7.2 (IN)
- net a1 renamed A1
- net A1: now also IC5.3 (I3), IC7.3 (IN)
- net a2 renamed A2
- net A2: now also IC5.4 (I4), IC7.4 (IN/PD)
- net a3 renamed A3
- net A3: now also IC5.5 (I5), IC7.5 (IN)
- net a4 renamed A4
- net A4: now also IC5.6 (I6), IC7.6 (IN)
- net a5 renamed A5
- net A5: now also IC7.7 (IN)
- net a6 renamed A6
- net A6: now also IC7.8 (IN)
- net a7 renamed A7
- net A7: now also IC7.9 (IN)
- net d0 renamed D0
- net D0: now also IC5.12 (IO8)
- net d1 renamed D1
- net D1: now also IC5.13 (IO7)
- net d2 renamed D2
- net D2: now also IC5.14 (IO6)
- net d3 renamed D3
- net D3: now also IC5.15 (IO5)
- net d4 renamed D4
- net D4: now also IC5.16 (IO4)
- net d5 renamed D5
- net D5: now also IC5.17 (I03)
- net d6 renamed D6
- net D6: now also IC5.18 (IO2)
- net d7 renamed D7
- net D7: now also IC5.19 (IO1)
- new net: OPTO1.8, R666.2
- new net: IC7.15 (I/O), TP1.1
- new net CS_ID: IC5.11 (I10/~{OE}), IC7.16 (I/O)
- new net Y3: IC7.20 (I/O)
- new net Y4: IC7.19 (I/O)
- new net ~{INT2}: IC2.7 (~{IRQ}), IC3.7 (~{IRQ}), IC4.7 (~{IRQ}), JP31.2 (B)
- no-connect marks 24 -> 21
Other:
- added sheet Untitled Sheet (untitled.kicad_sch)
- moved on the sheet: C11, C12, C2, CD1, CD10, CD11, CD2, CD4, CD5, CD7, CD8, D66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
